Commit message: Add environments

File: environments/environments_robot_task/robots/UR5/ur5.urdf (robot description, URDF)
Before this commit: robot ur5, 11 links, 10 joints
Joints:
- joint left_inner_finger_joint: origin xyz=0.0064 0 0.126 rpy=0 0 0 -> xyz=0.04 0 0.126 rpy=0 0 0; type prismatic -> fixed
- joint right_inner_finger_joint: origin xyz=-0.0064 0 0.126 rpy=0 0 3.1416 -> xyz=-0.04 0 0.126 rpy=0 0 3.1416; type prismatic -> fixed

Commit message: Make project installable

File: environments/environments_robot_task/robots/UR5/ur5.urdf (robot description, URDF)
Before this commit: robot ur5, 11 links, 10 joints
Links:
- link base_link: mass 0.0 -> 4.0

File: environments/environments_robot_task/robots/iiwa/iiwa.urdf (robot description, URDF)
Before this commit: robot lbr_iiwa, 12 links, 11 joints
Joints:
- joint left_inner_finger_joint: type prismatic -> fixed
- joint right_inner_finger_joint: origin xyz=-0.0064 0 0.126 rpy=0 0 3.1416 -> xyz=-0.04 0 0.126 rpy=0 0 3.1416; type prismatic -> fixed

Commit message: Add working version of UR5 IK

File: environments/environments_robot_task/robots/UR5/ur5.urdf (robot description, URDF)
Before this commit: robot ur5, 11 links, 10 joints
Joints:
- joint tcp: origin xyz=0.0 0.0 0.15 rpy=3.14159 0 -1.570796 -> xyz=0.0 0.0 0.15 rpy=0 0 0

Commit message: Add interactive demonstrator v2 - multi-step action imitation

File: environments/environments_robot_task/robots/UR5/ur5.urdf (robot description, URDF)
Before this commit: robot ur5, 11 links, 10 joints
Joints:
- joint elbow_joint: limit lower=0 upper=3.14159265359 effort=300.0 velocity=3.15 -> lower=-3.14159265359 upper=3.14159265359 effort=300.0 velocity=3.15
- joint shoulder_lift_joint: limit lower=-2.35619449019 upper=2.35619449019 effort=300.0 velocity=3.15 -> lower=-3.14159265359 upper=3.14159265359 effort=300.0 velocity=3.15
- joint shoulder_pan_joint: limit lower=-6.28318530718 upper=6.28318530718 effort=300.0 velocity=3.15 -> lower=-3.14159265359 upper=3.14159265359 effort=300.0 velocity=3.15
- joint wrist_1_joint: limit lower=-2.35619449019 upper=2.35619449019 effort=300.0 velocity=3.2 -> lower=-3.14159265359 upper=3.14159265359 effort=300.0 velocity=3.2
- joint wrist_2_joint: limit lower=-6.28318530718 upper=6.28318530718 effort=300.0 velocity=3.2 -> lower=-3.14159265359 upper=3.14159265359 effort=300.0 velocity=3.2
- joint wrist_3_joint: limit lower=-6.28318530718 upper=6.28318530718 effort=300.0 velocity=3.2 -> lower=-3.14159265359 upper=3.14159265359 effort=300.0 velocity=3.2
